Commit message: Add initial configuration and launch files for naviarm_bringup package

File: naviarm_description/urdf/naviarm_moveit_arm.xacro (robot description, xacro)
@@ -40,5 +40,5 @@
     <xacro:arg name="kinematics_suffix" default="" />
     <xacro:arg name="load_gazebo_plugin" default="true" />
-    <xacro:include filename="$(find autoserve_description)/urdf/autoserve.xacro" />
+    <link name="base_footprint" />
     <xacro:include filename="$(find xarm_description)/urdf/xarm_device_macro.xacro" />
     <xacro:xarm_device
