Commit message: Refactor code structure for improved readability and maintainability

File: naviarm_description/urdf/naviarm_ros_control.xacro (robot description, xacro)
@@ -89,5 +89,5 @@
             <state_interface name="velocity" />
         </joint>
-        <joint name="base2leftw">
+        <!-- <joint name="base2leftw">
             <command_interface name="velocity">
                 <param name="min">-10</param>
@@ -104,5 +104,5 @@
             <state_interface name="position" />
             <state_interface name="velocity" />
-        </joint>
+        </joint> -->
     </ros2_control>
 </robot>
